File: circuit/multicopter/motors.kicad_sch (KiCad schematic)
At the start: 36 parts, among them M1 Motor_DC, M2 Motor_DC, M3 Motor_DC, M4 Motor_DC, M5 Motor_DC, M6 Motor_DC, Q1 SQ2310CES, Q2 SQ2310CES, Q3 SQ2310CES, Q4 SQ2310CES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

Commit message: completed schematic.
Connections:
- net 0 renamed GND
Other:
- moved on the sheet: C2, D2, M2, Q2, R2, R4
