File: circuit/multicopter2/motors.kicad_sch (KiCad schematic)
At the start: 36 parts, among them M1 Motor_DC, M2 Motor_DC, M3 Motor_DC, M4 Motor_DC, M5 Motor_DC, M6 Motor_DC, Q1 SQ2310CES, Q2 SQ2310CES, Q3 SQ2310CES, Q4 SQ2310CES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

Commit message: added circuits.
Parts:
- removed C11: 22uF, Capacitor_SMD:C_0603_1608Metric, symbol Device:C_Small
- removed R16, R18: 100Ω, Resistor_SMD:R_0603_1608Metric, symbol Device:R
- removed R17, R19: 10kΩ, Resistor_SMD:R_0603_1608Metric, symbol Device:R
- added C6: 22uF, Capacitor_SMD:C_0603_1608Metric, symbol Device:C_Small
- added R10, R9: 100Ω, Resistor_SMD:R_0603_1608Metric, symbol Device:R
- added R11, R12: 10kΩ, Resistor_SMD:R_0603_1608Metric, symbol Device:R
- C1, C2, C3, C4, C5: Unit Price 85.8 -> 36.3
- D1, D2, D3, D4, D6, D7: Unit Price 62.7 -> 56.9
- M1, M2, M3, M4, M5, M6: footprint Connector_JST:JST_PH_S2B-PH-K_1x02_P2.00mm_Horizontal -> Connector_PinHeader_2.54mm:PinHeader_1x02_P2.54mm_Vertical; MANUFACTURER JST Sales America Inc. -> Adam Tech; Production Number S2B-PH-K-S -> PH1-02-UA; Purchase link https://www.digikey.jp/en/products/detail/jst-sales-america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 -> https://www.digikey.jp/ja/products/detail/adam-tech/PH1-02-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; Unit Price 15.04 -> 15
- Q1, Q2, Q3, Q4, Q5, Q6: Unit Price 77.6 -> 75.8
- R1, R2, R5, R6: Unit Price 16.5 -> 15.8
- R3, R4, R7, R8: Unit Price 23.1 -> 22.1
Connections:
- net +BATT: now also C6.1
- net GND: now also C6.2, R11.1, R12.1
- net motor3: now also R9.2; no longer R2.2
- net motor4: now also R2.2
- net motor6: now also R10.2
- net at Q6.1 (G): now also R10.1, R12.2
- net at Q5.1 (G): now also R11.2, R9.1
